File: INFERNO.kicad_sch (KiCad schematic)
At the start: 5 parts, among them J1 Conn_Coaxial_Small, J2 Micro_SD_Card, J3 Conn_01x05, U2 RFM95W-915S2, U3 SEN-13879

Commit message: finished mk1 design for production
Parts:
- added BZ1: CI12E-07T230-C-6, Buzzer_Beeper:Buzzer_15x7.5RM7.6, symbol Device:Buzzer
- added C1: 0.1uF, Capacitor_SMD:C_0603_1608Metric, symbol Device:C_Small
- added C2: 4.7uF, Capacitor_SMD:C_0603_1608Metric, symbol Device:C_Small
- added C3, C4, C5, C6, C7: 100nF, Capacitor_SMD:C_0603_1608Metric, symbol Device:C_Small
- added H1, H2, H3, H4: MountingHole, MountingHole:MountingHole_3.2mm_M3_ISO7380_Pad_TopBottom, symbol Mechanical:MountingHole
- added J10, J4, J5, J9: Conn_01x03, Connector_JST:JST_XH_B3B-XH-A_1x03_P2.50mm_Vertical, symbol Connector_Generic:Conn_01x03
- added J11, J6: Conn_01x03, Connector_PinSocket_2.54mm:PinSocket_1x03_P2.54mm_Vertical, symbol Connector_Generic:Conn_01x03
- added J12, J7: Conn_01x05, Connector_PinHeader_2.54mm:PinHeader_1x05_P2.54mm_Vertical, symbol Connector_Generic:Conn_01x05
- added J13: Conn_01x06, Connector_PinHeader_2.54mm:PinHeader_1x06_P2.54mm_Vertical, symbol Connector_Generic:Conn_01x06
- added J14: Conn_01x02, Connector_AMASS:AMASS_XT30PW-M_1x02_P2.50mm_Horizontal, symbol Connector_Generic:Conn_01x02
- added J15: Conn_01x02, TerminalBlock_Phoenix:TerminalBlock_Phoenix_MKDS-1,5-2-5.08_1x02_P5.08mm_Horizontal, symbol Connector_Generic:Conn_01x02
- added J17: Conn_01x02, Connector_PinSocket_2.54mm:PinSocket_1x02_P2.54mm_Vertical, symbol Connector_Generic:Conn_01x02
- added J8: Conn_01x14, Connector_PinHeader_2.54mm:PinHeader_1x14_P2.54mm_Vertical, symbol Connector_Generic:Conn_01x14
- added Q1: NMOS, Package_TO_SOT_SMD:SOT-323_SC-70, symbol Simulation_SPICE:NMOS
- added Q2: NMOS, Package_TO_SOT_SMD:TO-252-2, symbol Simulation_SPICE:NMOS
- added R1, R14, R15, R8, R9: 10k, Resistor_SMD:R_0603_1608Metric, symbol Device:R_Small
- added R10, R11, R12, R13: 20k, Resistor_SMD:R_0603_1608Metric, symbol Device:R_Small
- added R2: 100k, Resistor_SMD:R_0603_1608Metric, symbol Device:R_Small
- added R3: 4.7k, Resistor_SMD:R_0603_1608Metric, symbol Device:R
- added R4, R5: 10k, Resistor_SMD:R_0603_1608Metric, symbol Device:R
- added R6: 27k, Resistor_SMD:R_0603_1608Metric, symbol Device:R_Small
- added R7: 470, Resistor_SMD:R_0603_1608Metric, symbol Device:R_Small
- added SW1, SW2: SW_Push, Button_Switch_SMD:SW_SPST_B3S-1000, symbol Switch:SW_Push
- added U2: STM32F722RETx, Package_QFP:LQFP-64_10x10mm_P0.5mm, symbol MCU_ST_STM32F7:STM32F722RETx
- added Y1: ECS-2520MV-240-BN, Oscillator:Oscillator_SMD_ECS_2520MV-xxx-xx-4Pin_2.5x2.0mm, symbol Oscillator:ECS-2520MV-xxx-xx
- J1: renamed from J2; footprint Connector_Card:microSD_HC_Molex_47219-2001 -> Connector_Card:microSD_HC_Molex_104031-0811
- renumbered J1 to J2, U2 to U1
Connections:
- net +3V3: now also C3.1, C4.1, C5.1, C6.1, C7.1, J13.3 (Pin_3), J7.1 (Pin_1), J8.1 (Pin_1), R3.2, R4.2, R5.2, SW1.2, U2.1 (VBAT), U2.13 (VDDA), U2.19 (VDD), U2.32 (VDD), U2.48 (VDD), U2.64 (VDD), Y1.4 (VDD)
- net +5VA: now also J10.1 (Pin_1), J13.1 (Pin_1), J4.1 (Pin_1), J5.1 (Pin_1), J9.1 (Pin_1)
- net GNDREF: now also C1.2, C2.2, C3.2, C4.2, C5.2, C6.2, C7.2, J10.2 (Pin_2), J11.2 (Pin_2), J13.2 (Pin_2), J14.1 (Pin_1), J17.2 (Pin_2), J4.2 (Pin_2), J5.2 (Pin_2), J6.2 (Pin_2), J7.2 (Pin_2), J8.2 (Pin_2), J9.2 (Pin_2), Q1.3 (S), Q2.3 (S), R1.2, R10.2, R11.2, R12.2, R13.2, R2.1, R7.2, SW2.2, U2.12 (VSSA), U2.18 (VSS), U2.31 (VSS), U2.47 (VSS), U2.63 (VSS), Y1.2 (GND)
- net HX711_CLK: now also U2.2 (PC13)
- net HX711_DAT: now also U2.3 (PC14)
- net LoRa_CS: now also U2.27 (PB2)
- net LoRa_INT: now also U2.28 (PB10)
- net LoRa_RST: now also U2.29 (PB11)
- net MISO: now also J12.4 (Pin_4), R3.1, U2.22 (PA6)
- net MOSI: now also J12.3 (Pin_3), U2.23 (PA7)
- net SCK: now also J12.5 (Pin_5), U2.21 (PA5)
- net SDMMC_CK: now also U2.53 (PC12)
- net SDMMC_CMD: now also U2.54 (PD2)
- net SDMMC_D0: now also U2.39 (PC8)
- net SDMMC_D1: now also U2.40 (PC9)
- net SDMMC_D2: now also U2.51 (PC10)
- net SDMMC_D3: now also U2.52 (PC11)
- new net: J5.3 (Pin_3), R9.1
- new net: J10.3 (Pin_3), R15.1
- new net: C2.1, U2.30 (VCAP_1)
- new net: BZ1.2 (-), Q1.1 (D)
- new net: Q1.2 (G), U2.16 (PA2)
- new net: R1.1, SW1.1, U2.60 (BOOT0)
- new net: U2.5 (PH0), Y1.3 (OUT)
- new net: J4.3 (Pin_3), R8.1
- new net: J9.3 (Pin_3), R14.1
- new net +5VD: BZ1.1 (+), J11.1 (Pin_1), J6.1 (Pin_1)
- new net ALG1: J13.6 (Pin_6), U2.26 (PB1)
- new net ALG2: J13.5 (Pin_5), U2.25 (PB0)
- new net ALG3: J13.4 (Pin_4), U2.24 (PC4)
- new net CONT: R2.2, R6.1, U2.20 (PA4)
- new net HALL1: R12.1, R14.2, U2.10 (PC2)
- new net HALL2: R13.1, R15.2, U2.11 (PC3)
- new net LED: J17.1 (Pin_1), U2.38 (PC7)
- new net LIPO+: J14.2 (Pin_2), J15.2 (Pin_2)
- new net NRST: C1.1, J7.5 (Pin_5), SW2.1, U2.7 (NRST)
- new net PA10: J8.11 (Pin_11), U2.43 (PA10)
- new net PA11: J8.10 (Pin_10), U2.44 (PA11)
- new net PA12: J8.9 (Pin_9), U2.45 (PA12)
- new net PA15: J8.8 (Pin_8), U2.50 (PA15)
- new net PB12: J8.14 (Pin_14), U2.33 (PB12)
- new net PB13: J8.13 (Pin_13), U2.34 (PB13)
- new net PB3: J8.7 (Pin_7), U2.55 (PB3)
- new net PB4: J8.6 (Pin_6), U2.56 (PB4)
- new net PB5: J8.5 (Pin_5), U2.57 (PB5)
- new net PB8: J8.4 (Pin_4), U2.61 (PB8)
- new net PB9: J8.3 (Pin_3), U2.62 (PB9)
- new net PC6: J8.12 (Pin_12), U2.37 (PC6)
- new net PT1: R10.1, R8.2, U2.8 (PC0)
- new net PT2: R11.1, R9.2, U2.9 (PC1)
- new net PY-: J15.1 (Pin_1), Q2.2 (D), R6.2
- new net PYRO: Q2.1 (G), R7.1, U2.17 (PA3)
- new net SCL: J12.1 (Pin_1), R5.1, U2.58 (PB6)
- new net SDA: J12.2 (Pin_2), R4.1, U2.59 (PB7)
- new net SERVO1: J6.3 (Pin_3), U2.14 (PA0)
- new net SERVO2: J11.3 (Pin_3), U2.15 (PA1)
- new net SWCLK: J7.4 (Pin_4), U2.49 (PA14)
- new net SWDIO: J7.3 (Pin_3), U2.46 (PA13)
- new net USB_D+: U2.36 (PB15)
- new net USB_D-: U2.35 (PB14)
- no-connect marks 7 -> 12
Other:
- removed sheet Microcontroller
- note added: "voltage divide 5V to 3.3V for analog sense"
- moved on the sheet: J2, J3, U1, U3
