File: power.kicad_sch (KiCad schematic)
At the start: 16 parts, among them U4 TPSM86837RCGR, U5 LM2937xMP

Commit message: finished mk1 design for production
Parts:
- added C11: 0.33uF, Capacitor_SMD:C_0603_1608Metric, symbol Device:C_Small
- added C13: 0.1uF, Capacitor_SMD:C_0603_1608Metric, symbol Device:C_Small
- added D1: LED_RD, LED_SMD:LED_0603_1608Metric, symbol Device:LED
- added J16: USB_B_Micro, Connector_USB:USB_Micro-B_Amphenol_10118193-0001LF_Horizontal, symbol Connector:USB_B_Micro
- added R17: 470, Resistor_SMD:R_0603_1608Metric, symbol Device:R
- added U6: UA78M33QDCYRQ1, Package_TO_SOT_SMD:SOT-223-3_TabPin2, symbol Regulator_Linear:UA78M33QDCYRQ1
- C10: renamed from C17; footprint (none) -> Capacitor_SMD:C_0603_1608Metric
- C14: renamed from C8; footprint (none) -> Capacitor_SMD:C_0603_1608Metric
- C19: renamed from C9; footprint (none) -> Capacitor_SMD:C_0603_1608Metric
- R16: renamed from R2; footprint (none) -> Resistor_SMD:R_0603_1608Metric
- R18: renamed from R3; footprint (none) -> Resistor_SMD:R_0603_1608Metric
- R19: renamed from R4; footprint (none) -> Resistor_SMD:R_0603_1608Metric
- renumbered C16 to C12, C10 to C15, C13 to C16, C12 to C17, C11 to C18, C14 to C8, C15 to C9
Connections:
- net GNDREF: now also C11.2, C13.2, J16.5 (GND), R17.1, U6.2 (GND)
- net LIPO+: now also C11.1, U6.1 (IN)
- new net: D1.1 (K), R17.2
- new net +3V3: C13.1, D1.2 (A), U6.3 (OUT)
- new net USB_D+: J16.3 (D+)
- new net USB_D-: J16.2 (D-)
- no-connect marks 5 -> 8
